Commit message: gemelo digital funcionando sin las cajas

File: install/mi_pkg_python/share/mi_pkg_python/urdf/ensamblaje.urdf (robot description, URDF)
Before this commit: robot ensamblaje, 4 links, 3 joints
Joints:
- joint efector_joint: limit lower=-100.0 upper=100.0 effort=100 velocity=1.0 -> lower=-0.150 upper=0.150 effort=100 velocity=1.0

File: install/mi_pkg_python/share/mi_pkg_python/urdf/ensamblaje.urdf.xacro (robot description, xacro)
@@ -1,16 +1,17 @@
 <?xml version="1.0" encoding="utf-8"?>
 <robot xmlns:xacro="http://ros.org/wiki/xacro" name="ensamblaje_doble">
-  <xacro:property name="p1" value="robot1_"/>
-  <xacro:property name="p2" value="robot2_"/>
+  <xacro:property name="p1" value="r1_"/>
+  <xacro:property name="p2" value="r2_"/>
+  <xacro:property name="altura_montaje" value="0.1"/>
   <link name="world"/>
-  <joint name="world_to_robot1" type="fixed">
+  <joint name="world_to_r1" type="fixed">
     <parent link="world"/>
     <child link="${p1}base_link"/>
-    <origin xyz="0 0 0" rpy="0 0 0"/>
-  </joint>
-  <joint name="world_to_robot2" type="fixed">
+    <origin xyz="0 0 ${altura_montaje}" rpy="0 0 0"/>
+  </joint>
+  <joint name="world_to_r2" type="fixed">
     <parent link="world"/>
     <child link="${p2}base_link"/>
-    <origin xyz="0 0.63 0" rpy="0 0 0"/>
+    <origin xyz="0 0.63 ${altura_montaje}" rpy="0 0 0"/>
   </joint>
   <link name="${p1}base_link">
