Commit message: correcion, home con april tags

File: install/mi_pkg_python/share/mi_pkg_python/urdf/ensamblaje.urdf.xacro (robot description, xacro)
@@ -1,8 +1,18 @@
 <?xml version="1.0" encoding="utf-8"?>
-<robot xmlns:xacro="http://ros.org/wiki/xacro" name="ensamblaje">
-  <!-- Prefijo para instanciar el mismo robot varias veces -->
-  <xacro:arg name="prefix" default=""/>
-  <xacro:property name="prefix" value="$(arg prefix)"/>
-  <link name="${prefix}base_link">
+<robot xmlns:xacro="http://ros.org/wiki/xacro" name="ensamblaje_doble">
+  <xacro:property name="p1" value="robot1_"/>
+  <xacro:property name="p2" value="robot2_"/>
+  <link name="world"/>
+  <joint name="world_to_robot1" type="fixed">
+    <parent link="world"/>
+    <child link="${p1}base_link"/>
+    <origin xyz="0 0 0" rpy="0 0 0"/>
+  </joint>
+  <joint name="world_to_robot2" type="fixed">
+    <parent link="world"/>
+    <child link="${p2}base_link"/>
+    <origin xyz="0 0.63 0" rpy="0 0 0"/>
+  </joint>
+  <link name="${p1}base_link">
     <inertial>
       <origin xyz="-0.099514 0.0017046 0.043359" rpy="0 0 0"/>
@@ -16,16 +26,14 @@
         <mesh filename="package://mi_pkg_python/urdf/meshes/base_link.STL"/>
       </geometry>
-      <material name="">
-        <color rgba="0.75294 0.75294 0.75294 1"/>
-      </material>
-    </visual>
-    <collision>
-      <origin xyz="0 0 0" rpy="0 0 0"/>
-      <geometry>
-        <mesh filename="package://mi_pkg_python/urdf/meshes/base_link.STL"/>
-      </geometry>
-    </collision>
-  </link>
-  <link name="${prefix}brazo_link">
+      <material name=""><color rgba="0.75294 0.75294 0.75294 1"/></material>
+    </visual>
+    <collision>
+      <origin xyz="0 0 0" rpy="0 0 0"/>
+      <geometry>
+        <mesh filename="package://mi_pkg_python/urdf/meshes/base_link.STL"/>
+      </geometry>
+    </collision>
+  </link>
+  <link name="${p1}brazo_link">
     <inertial>
       <origin xyz="0.075309 -1.0471E-05 0.17304" rpy="0 0 0"/>
@@ -39,23 +47,21 @@
         <mesh filename="package://mi_pkg_python/urdf/meshes/brazo_link.STL"/>
       </geometry>
-      <material name="">
-        <color rgba="0.75294 0.75294 0.75294 1"/>
-      </material>
-    </visual>
-    <collision>
-      <origin xyz="0 0 0" rpy="0 0 0"/>
-      <geometry>
-        <mesh filename="package://mi_pkg_python/urdf/meshes/brazo_link.STL"/>
-      </geometry>
-    </collision>
-  </link>
-  <joint name="${prefix}brazo_joint" type="revolute">
+      <material name=""><color rgba="0.75294 0.75294 0.75294 1"/></material>
+    </visual>
+    <collision>
+      <origin xyz="0 0 0" rpy="0 0 0"/>
+      <geometry>
+        <mesh filename="package://mi_pkg_python/urdf/meshes/brazo_link.STL"/>
+      </geometry>
+    </collision>
+  </link>
+  <joint name="${p1}brazo_joint" type="revolute">
     <origin xyz="0 0 0" rpy="0 0 0"/>
-    <parent link="${prefix}base_link"/>
-    <child  link="${prefix}brazo_link"/>
+    <parent link="${p1}base_link"/>
+    <child  link="${p1}brazo_link"/>
     <axis xyz="0 0 1"/>
     <limit lower="-6.14" upper="6.14" effort="5.0" velocity="1.570"/>
   </joint>
-  <link name="${prefix}antebrazo_link">
+  <link name="${p1}antebrazo_link">
     <inertial>
       <origin xyz="0.12022 0.002532 0.013813" rpy="0 0 0"/>
@@ -69,23 +75,21 @@
         <mesh filename="package://mi_pkg_python/urdf/meshes/antebrazo_link.STL"/>
       </geometry>
-      <material name="">
-        <color rgba="0.75294 0.75294 0.75294 1"/>
-      </material>
-    </visual>
-    <collision>
-      <origin xyz="0 0 0" rpy="0 0 0"/>
-      <geometry>
-        <mesh filename="package://mi_pkg_python/urdf/meshes/antebrazo_link.STL"/>
-      </geometry>
-    </collision>
-  </link>
-  <joint name="${prefix}antebrazo_joint" type="revolute">
+      <material name=""><color rgba="0.75294 0.75294 0.75294 1"/></material>
+    </visual>
+    <collision>
+      <origin xyz="0 0 0" rpy="0 0 0"/>
+      <geometry>
+        <mesh filename="package://mi_pkg_python/urdf/meshes/antebrazo_link.STL"/>
+      </geometry>
+    </collision>
+  </link>
+  <joint name="${p1}antebrazo_joint" type="revolute">
     <origin xyz="0.20188 -0.00036684 0.15187" rpy="0 0 0"/>
-    <parent link="${prefix}brazo_link"/>
-    <child  link="${prefix}antebrazo_link"/>
+    <parent link="${p1}brazo_link"/>
+    <child  link="${p1}antebrazo_link"/>
     <axis xyz="0 0 1"/>
     <limit lower="-6.14" upper="6.14" effort="5" velocity="1.570"/>
   </joint>
-  <link name="${prefix}efector_link">
+  <link name="${p1}efector_link">
     <inertial>
       <origin xyz="-0.00019941 3.011E-05 -0.092013" rpy="0 0 0"/>
@@ -99,21 +103,124 @@
         <mesh filename="package://mi_pkg_python/urdf/meshes/efector_link.STL"/>
       </geometry>
-      <material name="">
-        <color rgba="0.75294 0.75294 0.75294 1"/>
-      </material>
-    </visual>
-    <collision>
-      <origin xyz="0 0 0" rpy="0 0 0"/>
-      <geometry>
-        <mesh filename="package://mi_pkg_python/urdf/meshes/efector_link.STL"/>
-      </geometry>
-    </collision>
-  </link>
-  <joint name="${prefix}efector_joint" type="prismatic">
+      <material name=""><color rgba="0.75294 0.75294 0.75294 1"/></material>
+    </visual>
+    <collision>
+      <origin xyz="0 0 0" rpy="0 0 0"/>
+      <geometry>
+        <mesh filename="package://mi_pkg_python/urdf/meshes/efector_link.STL"/>
+      </geometry>
+    </collision>
+  </link>
+  <joint name="${p1}efector_joint" type="prismatic">
     <origin xyz="0.20445 0.001 +0.13418" rpy="3.1416 0 0"/>
-    <parent link="${prefix}antebrazo_link"/>
-    <child  link="${prefix}efector_link"/>
+    <parent link="${p1}antebrazo_link"/>
+    <child  link="${p1}efector_link"/>
     <axis xyz="0 0 1"/>
     <limit lower="-0.15" upper="0.15" effort="0" velocity="0.05"/>
   </joint>
+  <link name="${p2}base_link">
+    <inertial>
+      <origin xyz="-0.099514 0.0017046 0.043359" rpy="0 0 0"/>
+      <mass value="1.395"/>
+      <inertia ixx="0.0019998" ixy="-5.6235E-07" ixz="-0.00017151"
+               iyy="0.004182" iyz="-8.2856E-07" izz="0.0049989"/>
+    </inertial>
+    <visual>
+      <origin xyz="0 0 0" rpy="0 0 0"/>
+      <geometry>
+        <mesh filename="package://mi_pkg_python/urdf/meshes/base_link.STL"/>
+      </geometry>
+      <material name=""><color rgba="0.75294 0.75294 0.75294 1"/></material>
+    </visual>
+    <collision>
+      <origin xyz="0 0 0" rpy="0 0 0"/>
+      <geometry>
+        <mesh filename="package://mi_pkg_python/urdf/meshes/base_link.STL"/>
+      </geometry>
+    </collision>
+  </link>
+  <link name="${p2}brazo_link">
+    <inertial>
+      <origin xyz="0.075309 -1.0471E-05 0.17304" rpy="0 0 0"/>
+      <mass value="0.46473"/>
+      <inertia ixx="0.00018478" ixy="2.9848E-09" ixz="-8.9803E-07"
+               iyy="0.0015038" iyz="-1.2762E-08" izz="0.0014571"/>
+    </inertial>
+    <visual>
+      <origin xyz="0 0 0" rpy="0 0 0"/>
+      <geometry>
+        <mesh filename="package://mi_pkg_python/urdf/meshes/brazo_link.STL"/>
+      </geometry>
+      <material name=""><color rgba="0.75294 0.75294 0.75294 1"/></material>
+    </visual>
+    <collision>
+      <origin xyz="0 0 0" rpy="0 0 0"/>
+      <geometry>
+        <mesh filename="package://mi_pkg_python/urdf/meshes/brazo_link.STL"/>
+      </geometry>
+    </collision>
+  </link>
+  <joint name="${p2}brazo_joint" type="revolute">
+    <origin xyz="0 0 0" rpy="0 0 0"/>
+    <parent link="${p2}base_link"/>
+    <child  link="${p2}brazo_link"/>
+    <axis xyz="0 0 1"/>
+    <limit lower="-6.14" upper="6.14" effort="5.0" velocity="1.570"/>
+  </joint>
+  <link name="${p2}antebrazo_link">
+    <inertial>
+      <origin xyz="0.12022 0.002532 0.013813" rpy="0 0 0"/>
+      <mass value="0.33783"/>
+      <inertia ixx="9.4347E-05" ixy="-3.4378E-06" ixz="-4.6981E-05"
+               iyy="0.0013614" iyz="-1.7572E-06" izz="0.0013587"/>
+    </inertial>
+    <visual>
+      <origin xyz="0 0 0" rpy="0 0 0"/>
+      <geometry>
+        <mesh filename="package://mi_pkg_python/urdf/meshes/antebrazo_link.STL"/>
+      </geometry>
+      <material name=""><color rgba="0.75294 0.75294 0.75294 1"/></material>
+    </visual>
+    <collision>
+      <origin xyz="0 0 0" rpy="0 0 0"/>
+      <geometry>
+        <mesh filename="package://mi_pkg_python/urdf/meshes/antebrazo_link.STL"/>
+      </geometry>
+    </collision>
+  </link>
+  <joint name="${p2}antebrazo_joint" type="revolute">
+    <origin xyz="0.20188 -0.00036684 0.15187" rpy="0 0 0"/>
+    <parent link="${p2}brazo_link"/>
+    <child  link="${p2}antebrazo_link"/>
+    <axis xyz="0 0 1"/>
+    <limit lower="-6.14" upper="6.14" effort="5" velocity="1.570"/>
+  </joint>
+  <link name="${p2}efector_link">
+    <inertial>
+      <origin xyz="-0.00019941 3.011E-05 -0.092013" rpy="0 0 0"/>
+      <mass value="0.064572"/>
+      <inertia ixx="9.9025E-05" ixy="1.0267E-11" ixz="4.8235E-07"
+               iyy="9.4422E-05" iyz="-1.0234E-08" izz="7.2977E-06"/>
+    </inertial>
+    <visual>
+      <origin xyz="0 0 0" rpy="0 0 0"/>
+      <geometry>
+        <mesh filename="package://mi_pkg_python/urdf/meshes/efector_link.STL"/>
+      </geometry>
+      <material name=""><color rgba="0.75294 0.75294 0.75294 1"/></material>
+    </visual>
+    <collision>
+      <origin xyz="0 0 0" rpy="0 0 0"/>
+      <geometry>
+        <mesh filename="package://mi_pkg_python/urdf/meshes/efector_link.STL"/>
+      </geometry>
+    </collision>
+  </link>
+  <joint name="${p2}efector_joint" type="prismatic">
+    <origin xyz="0.20445 0.001 +0.13418" rpy="3.1416 0 0"/>
+    <parent link="${p2}antebrazo_link"/>
+    <child  link="${p2}efector_link"/>
+    <axis xyz="0 0 1"/>
+    <limit lower="-0.15" upper="0.15" effort="0" velocity="0.05"/>
+  </joint>
 </robot>

Commit message: actualizacion del gemelo digital y puntos de scara 1,2

File: install/mi_pkg_python/share/mi_pkg_python/urdf/ensamblaje.urdf.xacro (robot description, xacro)
@@ -1,17 +1,75 @@
 <?xml version="1.0" encoding="utf-8"?>
-<robot xmlns:xacro="http://ros.org/wiki/xacro" name="ensamblaje_doble">
+<robot xmlns:xacro="http://ros.org/wiki/xacro" name="ensamblaje_doble_con_banda">
   <xacro:property name="p1" value="r1_"/>
   <xacro:property name="p2" value="r2_"/>
-  <xacro:property name="altura_montaje" value="0.1"/>
+  <xacro:property name="altura_montaje" value="0.25"/>
   <link name="world"/>
   <joint name="world_to_r1" type="fixed">
     <parent link="world"/>
     <child link="${p1}base_link"/>
-    <origin xyz="0 0 ${altura_montaje}" rpy="0 0 0"/>
+    <origin xyz="0.10 0 ${altura_montaje}" rpy="0 0 0"/>
   </joint>
   <joint name="world_to_r2" type="fixed">
     <parent link="world"/>
     <child link="${p2}base_link"/>
-    <origin xyz="0 0.63 ${altura_montaje}" rpy="0 0 0"/>
+    <origin xyz="0.10 0.63 ${altura_montaje}" rpy="0 0 0"/>
+  </joint>
+  <joint name="world_to_banda" type="fixed">
+    <parent link="world"/>
+    <child link="banda_base_link"/>
+    <origin xyz="0 0 0" rpy="0 0 0"/>
+  </joint>
+  <link name="banda_base_link">
+    <inertial>
+      <origin xyz="0.532375158645714 -0.00125118407977348 -0.0614188025075904" rpy="0 0 0" />
+      <mass value="3.53485764601871" />
+      <inertia ixx="0.010351026660149" ixy="-1.61847933564091E-05" ixz="-8.83817332567959E-07"
+               iyy="0.341234100404499" iyz="4.24067313651221E-07" izz="0.35088951437036" />
+    </inertial>
+    <visual>
+      <origin xyz="0.4 -0.2 0" rpy="0 0 1.5708" />
+      <geometry>
+        <mesh filename="package://mi_pkg_python/urdf/meshes/banda_base_link.STL" />
+      </geometry>
+      <material name="">
+        <color rgba="0.592156862745098 0.117647058823529 0 1" />
+      </material>
+    </visual>
+    <collision>
+      <origin xyz="0 0 0" rpy="0 0 0" />
+      <geometry>
+        <mesh filename="package://mi_pkg_python/urdf/meshes/banda_base_link.STL" />
+      </geometry>
+    </collision>
+  </link>
+  <link name="banda_link">
+    <inertial>
+      <origin xyz="0.54526 -1.9429E-16 0" rpy="0 0 0" />
+      <mass value="0.5909" />
+      <inertia ixx="0.00061358" ixy="-1.2903E-17" ixz="1.5247E-19"
+               iyy="0.059266" iyz="-1.2783E-20" izz="0.059878" />
+    </inertial>
+    <visual>
+      <origin xyz="0.4 -0.2 0" rpy="0 0 1.5708" />
+      <geometry>
+        <mesh filename="package://mi_pkg_python/urdf/meshes/banda_link.STL" />
+      </geometry>
+      <material name="">
+        <color rgba="0.59216 0.11765 0 1" />
+      </material>
+    </visual>
+    <collision>
+      <origin xyz="0 0 0" rpy="0 0 0" />
+      <geometry>
+        <mesh filename="package://mi_pkg_python/urdf/meshes/banda_link.STL" />
+      </geometry>
+    </collision>
+  </link>
+  <joint name="banda_joint" type="prismatic">
+    <origin xyz="0 0 0" rpy="0 0 0" />
+    <parent link="banda_base_link" />
+    <child link="banda_link" />
+    <axis xyz="1 0 0" />
+    <limit lower="0" upper="0" effort="0" velocity="0" />
   </joint>
   <link name="${p1}base_link">
